File: kicad/RetroWiFiModem.kicad_pcb (KiCad board)
At the start: 2 copper layers, 100 x 66.1 mm, 35 parts, among them CON1 BarrelJack_Horizontal, P1 CONN_02X05, U1 MAX3237CAI+, U2 74HCT245, U3 74HC32, U4 L4931CZ33-AP, U5 WeMos_mini, U6 DFPlayer_Mini

Commit message: Sync Repo
Parts:
- removed D9: 1N4148, modules:D_DO-35_SOD27_P7.62mm_Horizontal
- removed LS1: Speaker, modules:PinHeader_1x02_P2.54mm_Vertical
- removed R10: 10K, footprints:R3
- removed U6: DFPlayer_Mini, modules:DFPlayerMini
- added R2: 560R, Resistor_THT:R_Axial_DIN0204_L3.6mm_D1.6mm_P7.62mm_Horizontal, F.Cu at (194.8, 124.2)
- added R3: 560R, Resistor_THT:R_Axial_DIN0204_L3.6mm_D1.6mm_P7.62mm_Horizontal, F.Cu at (194.8, 117.6)
- added R4: 560R, Resistor_THT:R_Axial_DIN0204_L3.6mm_D1.6mm_P7.62mm_Horizontal, F.Cu at (194.8, 111.0)
- added R5: 560R, Resistor_THT:R_Axial_DIN0204_L3.6mm_D1.6mm_P7.62mm_Horizontal, F.Cu at (194.8, 104.4)
- added R6: 560R, Resistor_THT:R_Axial_DIN0204_L3.6mm_D1.6mm_P7.62mm_Horizontal, F.Cu at (194.8, 97.8)
- added R7: 560R, Resistor_THT:R_Axial_DIN0204_L3.6mm_D1.6mm_P7.62mm_Horizontal, F.Cu at (194.8, 91.2)
- added R8: 560R, Resistor_THT:R_Axial_DIN0204_L3.6mm_D1.6mm_P7.62mm_Horizontal, F.Cu at (194.8, 84.6)
- C1, C2, C3, C4, C5, C7, C8: footprint modules:C_Disc_D3_P2.5 -> Capacitor_THT:C_Disc_D3.0mm_W2.0mm_P2.50mm
- C6: footprint footprints:R3 -> Capacitor_THT:C_Disc_D5.0mm_W2.5mm_P5.00mm
- CON1: value BarrelJack_Horizontal -> BARREL_JACK; footprint footprints:BarrelJack_Horizontal -> Connector_BarrelJack:BarrelJack_Horizontal
- D1, D2, D3, D4, D5, D6, D7, D8: footprint modules:LED-3MM -> LED_THT:LED_D3.0mm
- H1, H2, H3, H4, H5, H6: footprint footprints:MountingHole_3.2mm -> MountingHole:MountingHole_3.2mm_M3
- P1: footprint modules:IDC_Header_Straight_10pins -> Connector_IDC:IDC-Header_2x05_P2.54mm_Vertical
- R1: footprint modules:DIP-16_W7.62mm_LongPads -> Resistor_THT:R_Axial_DIN0204_L3.6mm_D1.6mm_P7.62mm_Horizontal
- R9: footprint footprints:R3 -> Resistor_THT:R_Axial_DIN0204_L3.6mm_D1.6mm_P7.62mm_Horizontal
- U1: value MAX3237CAI+ -> 74HC245; footprint modules:SOIC-28W_7.5x17.9mm_Pitch1.27mm -> Package_DIP:DIP-20_W7.62mm
- U2: value 74HCT245 -> MAX3232; footprint modules:SOIC-20W_7.5x12.8mm_P1.27mm -> Package_DIP:DIP-16_W7.62mm
- U3: footprint modules:SOIC-14_3.9x8.7mm_P1.27mm -> Package_DIP:DIP-14_W7.62mm
- U4: value L4931CZ33-AP -> LP2950ACZ-3.3; footprint modules:TO-92_Inline_Wide -> Package_TO_SOT_THT:TO-92L_Inline_Wide
- U5: value WeMos_mini -> WeMos_D1_mini; footprint modules:wemos-d1-mini-with-pin-header-and-connector -> RetroWiFiModem-footprints:wemos-d1-mini
- moved U2 63.1 mm to (142.2, 78.7)
- moved H2 61.1 mm to (119.5, 132.0)
- moved U1 56.0 mm to (181.6, 128.3), turned to 180 degrees
- moved H5 55.1 mm to (189.4, 85.8)
- moved D1 46.2 mm to (205.7, 130.7)
- moved D8 46.2 mm to (205.7, 84.5)
- moved H4 40.0 mm to (159.4, 132.0)
- moved D2 33.0 mm to (205.7, 124.1)
- moved D7 33.0 mm to (205.7, 91.1)
- moved R9 31.2 mm to (162.6, 90.2), turned to 270 degrees
- moved H3 30.0 mm to (159.4, 85.8)
- moved C7 25.8 mm to (180.3, 86.4), turned to 90 degrees
- moved U3 23.0 mm to (166.4, 97.8), turned to 90 degrees
- moved R1 22.2 mm to (194.8, 130.7)
- moved U4 20.4 mm to (176.5, 86.4), turned to 90 degrees
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Connections:
- C3 pad 1: +3V3 -> Net-(C3-Pad1)
- C3 pad 2: Net-(C3-Pad2) -> GND
- CON1 pad 3: unconnected-(CON1-Pad3) -> Net-(CON1-Pad3)
- P1 pad 10: unconnected-(P1-Pad10) -> Net-(P1-Pad10)
- R1 pad 2: Net-(R1-Pad2) -> Net-(D1-Pad1)
- U1 pad 1: Net-(C1-Pad1) -> GND
- U1 pad 10: Net-(P1-Pad2) -> GND
- U1 pad 11: Net-(P1-Pad7) -> Net-(U1-Pad11)
- U1 pad 12: Net-(P1-Pad8) -> GND
- U1 pad 13: Net-(R9-Pad2) -> Net-(U1-Pad13)
- U1 pad 14: +3V3 -> Net-(U1-Pad14)
- U1 pad 15: GND -> Net-(U1-Pad15)
- U1 pad 16: unconnected-(U1-Pad16) -> Net-(U1-Pad16)
- U1 pad 19: Net-(U1-Pad19) -> GND
- U1 pad 2: GND -> Net-(R1-Pad1)
- U1 pad 20: Net-(U1-Pad20) -> +5V
- U1 pad 3: Net-(C1-Pad2) -> Net-(R2-Pad1)
- U1 pad 4: Net-(C2-Pad1) -> Net-(R3-Pad1)
- U1 pad 5: Net-(P1-Pad3) -> Net-(R4-Pad1)
- U1 pad 6: Net-(P1-Pad6) -> Net-(R5-Pad1)
- U1 pad 7: Net-(P1-Pad1) -> Net-(R6-Pad1)
- U1 pad 8: Net-(P1-Pad5) -> Net-(R7-Pad1)
- U1 pad 9: Net-(P1-Pad4) -> Net-(R8-Pad1)
- U2 pad 1: +5V -> Net-(C6-Pad1)
- U2 pad 10: GND -> Net-(U1-Pad17)
- U2 pad 11: Net-(R1-Pad8) -> Net-(U1-Pad14)
- U2 pad 12: Net-(R1-Pad7) -> Net-(U1-Pad13)
- U2 pad 13: Net-(R1-Pad6) -> Net-(P1-Pad5)
- U2 pad 14: Net-(R1-Pad5) -> Net-(P1-Pad3)
- U2 pad 15: Net-(R1-Pad4) -> GND
- U2 pad 16: Net-(R1-Pad3) -> +3V3
- U2 pad 2: Net-(U1-Pad19) -> Net-(C2-Pad1)
- U2 pad 3: Net-(U1-Pad18) -> Net-(C6-Pad2)
- U2 pad 4: Net-(U1-Pad21) -> Net-(C1-Pad1)
- U2 pad 5: Net-(U1-Pad24) -> Net-(C1-Pad2)
- U2 pad 6: Net-(U1-Pad17) -> Net-(C3-Pad1)
- U2 pad 7: Net-(U1-Pad22) -> Net-(P1-Pad6)
- U2 pad 8: Net-(U1-Pad23) -> Net-(P1-Pad4)
- U2 pad 9: Net-(U1-Pad20) -> Net-(U1-Pad18)
- U3 pad 11: unconnected-(U3-Pad11) -> Net-(U3-Pad11)
- U3 pad 3: Net-(U1-Pad24) -> Net-(U1-Pad14)
- U3 pad 6: unconnected-(U3-Pad6) -> Net-(U3-Pad6)
- U3 pad 8: unconnected-(U3-Pad8) -> Net-(U3-Pad8)
- U5 pad 10: unconnected-(U5-Pad10) -> Net-(U5-Pad10)
- U5 pad 13: Net-(U1-Pad17) -> Net-(U1-Pad15)
- U5 pad 14: Net-(U1-Pad20) -> Net-(U1-Pad18)
- U5 pad 15: Net-(U1-Pad23) -> Net-(U1-Pad17)
- U5 pad 16: unconnected-(U5-Pad16) -> Net-(U5-Pad16)
- U5 pad 4: Net-(U1-Pad18) -> Net-(U5-Pad4)
- U5 pad 5: Net-(U1-Pad19) -> Net-(U1-Pad11)
- U5 pad 6: Net-(U1-Pad22) -> Net-(U1-Pad16)
- U5 pad 7: Net-(U1-Pad21) -> Net-(U1-Pad13)
- U5 pad 9: unconnected-(U5-Pad9) -> Net-(U5-Pad9)
Routing:
- net Net-(U1-Pad23): track 81.4 -> 0.00 mm, vias 4 -> 0
- net Net-(U1-Pad24): track 79.7 -> 0.00 mm, vias 4 -> 0
- net Net-(U1-Pad20): track 78.4 -> 0.00 mm, vias 4 -> 0
- net Net-(U1-Pad21): track 77.8 -> 0.00 mm, vias 5 -> 0
- net Net-(U1-Pad22): track 75.2 -> 0.00 mm, vias 5 -> 0
- net Net-(U1-Pad13): track 0.00 -> 63.1 mm, vias 0 -> 8
- net Net-(U1-Pad19): track 61.8 -> 0.00 mm, vias 1 -> 0
- net +3V3: track 113.6 -> 55.8 mm, vias 5 -> 0
- net Net-(U5-Pad3): track 56.7 -> 0.00 mm, vias 2 -> 0
- net Net-(U1-Pad14): track 0.00 -> 42.7 mm, vias 0 -> 2
- net Net-(U1-Pad11): track 0.00 -> 41.9 mm, vias 0 -> 2
- net Net-(U5-Pad11): track 33.7 -> 0.00 mm
- net Net-(R9-Pad2): track 57.6 -> 24.6 mm, vias 4 -> 0
- net Net-(R1-Pad6): track 32.0 -> 0.00 mm, vias 1 -> 0
- net Net-(U1-Pad15): track 0.00 -> 30.9 mm
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- removed copper zone on F.Cu, net GND
Other:
- board size 100 x 66.1 mm -> 102.5 x 66.1 mm
- net class Default added: clearance 0.2, trace_width 0.38, via_dia 1.4, via_drill 0.9
- net class Power added: clearance 0.3, trace_width 0.5, via_dia 1.4, via_drill 0.9
- rule pad_to_mask_clearance: 0 -> 0.2
- board text added: "Retro WiFi Modem PCB 0.3 March 24, 2020"
- board text removed: "CD"
- board text removed: "CS"
- board text removed: "JLCJLCJLCJLC"
- board text removed: "MR"
- board text removed: "RD"
- board text removed: "RI"
- board text removed: "RS"
- board text removed: "Retro WiFi Modem PCB 2.2 April 17, 2024"
- board text removed: "SD"
- board text removed: "TR"
